File: hardware/kicad/emon36/emon36.kicad_pcb (KiCad board)
At the start: 4 copper layers, 80 x 99.1 mm, 258 parts, among them J1 Barrel_Jack, J10 STX-4335-5BGP-S1, J11 STX-4335-5BGP-S1, J12 STX-4335-5BGP-S1, J13 STX-4335-5BGP-S1, J14 STX-4335-5BGP-S1, J15 STX-4335-5BGP-S1, J2 STX-4335-5BGP-S1, J3 STX-4335-5BGP-S1, J37 USB_B_Micro, J4 STX-4335-5BGP-S1, J5 STX-4335-5BGP-S1, J6 STX-4335-5BGP-S1, J7 STX-4335-5BGP-S1, J8 STX-4335-5BGP-S1, J9 STX-4335-5BGP-S1, SW1 SW_MEC_5E, SW2 SW_MEC_5E, SW3 SW_MEC_5E, SW4 SW_MEC_5E, SW5 SW_MEC_5E, SW6 SW_MEC_5E, U1 ESP32-C3-WROOM-02-N4, U8 TPS54233

Commit message: Another major schematics/PCB iteration. Added decoupling caps, interrupts, etc. Improved power system. Added clock.
Parts:
- removed SW6: SW_MEC_5E, Button_Switch_SMD:SW_Push_1P1T_NO_6x6mm_H13mm
- added C100: 4.7uF, Capacitor_SMD:C_0603_1608Metric, F.Cu at (96.4, 132.5)
- added C101: 0.22uF, Capacitor_SMD:C_0603_1608Metric, F.Cu at (89.6, 126.0)
- added C102: 0.1uF, Capacitor_SMD:C_0603_1608Metric, F.Cu at (98.3, 132.7)
- added C103: 22nF, Capacitor_SMD:C_0603_1608Metric, F.Cu at (93.0, 135.6)
- added C104: 22nF, Capacitor_SMD:C_0603_1608Metric, F.Cu at (96.4, 129.0)
- added C105: 4.7uF, Capacitor_SMD:C_0603_1608Metric, F.Cu at (89.5, 137.4)
- added C106: 0.22uF, Capacitor_SMD:C_0603_1608Metric, F.Cu at (89.5, 135.6)
- added C107: 22nF, Capacitor_SMD:C_0603_1608Metric, F.Cu at (49.2, 58.1)
- added C108: 22nF, Capacitor_SMD:C_0603_1608Metric, F.Cu at (49.2, 53.6)
- added C109: 22nF, Capacitor_SMD:C_0603_1608Metric, F.Cu at (49.1, 49.3)
- added C110: 22nF, Capacitor_SMD:C_0603_1608Metric, F.Cu at (49.2, 70.8)
- added C111: 22nF, Capacitor_SMD:C_0603_1608Metric, F.Cu at (49.2, 66.6)
- added C112: 22nF, Capacitor_SMD:C_0603_1608Metric, F.Cu at (49.2, 62.6)
- added C113: 4.7uF, Capacitor_SMD:C_0603_1608Metric, F.Cu at (58.9, 69.6)
- added C114: 4.7uF, Capacitor_SMD:C_0603_1608Metric, F.Cu at (55.0, 63.0)
- added C115: 0.22uF, Capacitor_SMD:C_0603_1608Metric, F.Cu at (61.9, 69.6)
- added C116: 0.1uF, Capacitor_SMD:C_0603_1608Metric, F.Cu at (53.1, 62.9)
- added C117: 22nF, Capacitor_SMD:C_0603_1608Metric, F.Cu at (58.4, 60.0)
- added C118: 22nF, Capacitor_SMD:C_0603_1608Metric, F.Cu at (55.0, 66.6)
- added C119: 4.7uF, Capacitor_SMD:C_0603_1608Metric, F.Cu at (61.9, 58.2)
- added C120: 0.22uF, Capacitor_SMD:C_0603_1608Metric, F.Cu at (61.9, 60.0)
- added D4: ABS6, Diode_SMD:Diode_Bridge_Diotec_ABS, F.Cu at (76.1, 128.5)
- added D5: B240, Diode_SMD:D_SMB, F.Cu at (137.9, 7.07)
- added J16: STX-4335-5BGP-S1, Connector_Audio:STX-4335-5BGP-S1_KYC, B.Cu at (34.8, 66.6)
- added JP1: SolderJumper_3_Bridged12, Jumper:SolderJumper-3_P1.3mm_Bridged12_RoundedPad1.0x1.5mm, F.Cu at (135.8, 18.6)
- added JP2: SolderJumper_3_Bridged12, Jumper:SolderJumper-3_P1.3mm_Bridged12_RoundedPad1.0x1.5mm, F.Cu at (141.4, 20.0)
- added JP3: Jumper_3_Bridged12, Connector_PinHeader_2.54mm:PinHeader_1x03_P2.54mm_Vertical, F.Cu at (126.8, 6.62)
- added JP4: Jumper_3_Bridged12, Connector_PinHeader_2.54mm:PinHeader_1x03_P2.54mm_Vertical, F.Cu at (131.4, 6.62)
- added MH1: MountingHole, MountingHole:MountingHole_2.7mm_M2.5, F.Cu at (145.6, 7.77)
- added MH2: MountingHole, MountingHole:MountingHole_2.7mm_M2.5, F.Cu at (152.5, 7.77)
- added MH3: MountingHole, MountingHole:MountingHole_2.7mm_M2.5, F.Cu at (137.2, 13.3)
- added MH4: MountingHole, MountingHole:MountingHole_2.7mm_M2.5, F.Cu at (144.2, 14.7)
- added NT1: NetTie_2, NetTie:NetTie-2_SMD_Pad0.5mm, F.Cu at (55.1, 85.6)
- added NT10: NetTie_2, NetTie:NetTie-2_SMD_Pad0.5mm, F.Cu at (98.1, 110.2)
- added NT11: NetTie_2, NetTie:NetTie-2_SMD_Pad0.5mm, F.Cu at (96.4, 135.6)
- added NT12: NetTie_2, NetTie:NetTie-2_SMD_Pad0.5mm, F.Cu at (98.2, 135.6)
- added NT13: NetTie_2, NetTie:NetTie-2_SMD_Pad0.5mm, F.Cu at (55.0, 60.0)
- added NT14: NetTie_2, NetTie:NetTie-2_SMD_Pad0.5mm, F.Cu at (53.3, 60.0)
- added NT2: NetTie_2, NetTie:NetTie-2_SMD_Pad0.5mm, F.Cu at (53.3, 85.6)
- added NT3: NetTie_2, NetTie:NetTie-2_SMD_Pad0.5mm, F.Cu at (55.2, 110.8)
- added NT4: NetTie_2, NetTie:NetTie-2_SMD_Pad0.5mm, F.Cu at (53.5, 110.8)
- added NT5: NetTie_2, NetTie:NetTie-2_SMD_Pad0.5mm, F.Cu at (96.3, 58.9)
- added NT6: NetTie_2, NetTie:NetTie-2_SMD_Pad0.5mm, F.Cu at (98.1, 58.9)
- added NT7: NetTie_2, NetTie:NetTie-2_SMD_Pad0.5mm, F.Cu at (96.4, 84.6)
- added NT8: NetTie_2, NetTie:NetTie-2_SMD_Pad0.5mm, F.Cu at (98.2, 84.6)
- added NT9: NetTie_2, NetTie:NetTie-2_SMD_Pad0.5mm, F.Cu at (96.3, 110.2)
- added R125: 499, Resistor_SMD:R_0603_1608Metric, F.Cu at (100.2, 112.0)
- added R126: 499, Resistor_SMD:R_0603_1608Metric, F.Cu at (100.2, 116.6)
- added R127: 499, Resistor_SMD:R_0603_1608Metric, F.Cu at (100.2, 120.9)
- added R128: 499, Resistor_SMD:R_0603_1608Metric, F.Cu at (100.2, 99.3)
- added R129: 499, Resistor_SMD:R_0603_1608Metric, F.Cu at (100.2, 103.6)
- added R130: 499, Resistor_SMD:R_0603_1608Metric, F.Cu at (100.2, 107.6)
- added R131: 1k, Resistor_SMD:R_0603_1608Metric, F.Cu at (93.1, 112.0)
- added R132: 1k, Resistor_SMD:R_0603_1608Metric, F.Cu at (98.1, 103.6)
- added R133: 22, Resistor_SMD:R_0603_1608Metric, F.Cu at (86.1, 107.1)
- added R134: RB, Resistor_SMD:R_0603_1608Metric, F.Cu at (109.5, 143.6)
- added R135: RB, Resistor_SMD:R_0603_1608Metric, F.Cu at (114.3, 143.2)
- added R136: RB, Resistor_SMD:R_0603_1608Metric, F.Cu at (119.4, 140.7)
- added R137: RB, Resistor_SMD:R_0603_1608Metric, F.Cu at (109.5, 130.0)
- added R138: RB, Resistor_SMD:R_0603_1608Metric, F.Cu at (114.1, 130.3)
- added R139: RB, Resistor_SMD:R_0603_1608Metric, F.Cu at (119.1, 131.1)
- added R140: 1k, Resistor_SMD:R_0603_1608Metric, F.Cu at (104.2, 137.4)
- added R141: 1k, Resistor_SMD:R_0603_1608Metric, F.Cu at (104.2, 141.9)
- added R142: 1k, Resistor_SMD:R_0603_1608Metric, F.Cu at (104.2, 146.3)
- added R143: 1k, Resistor_SMD:R_0603_1608Metric, F.Cu at (104.2, 124.7)
- added R144: 1k, Resistor_SMD:R_0603_1608Metric, F.Cu at (104.2, 129.0)
- added R145: 1k, Resistor_SMD:R_0603_1608Metric, F.Cu at (104.2, 133.0)
- added R146: 499, Resistor_SMD:R_0603_1608Metric, F.Cu at (100.3, 137.4)
- added R147: 499, Resistor_SMD:R_0603_1608Metric, F.Cu at (100.3, 142.0)
- added R148: 499, Resistor_SMD:R_0603_1608Metric, F.Cu at (100.3, 146.3)
- added R149: 499, Resistor_SMD:R_0603_1608Metric, F.Cu at (100.3, 124.7)
- added R150: 499, Resistor_SMD:R_0603_1608Metric, F.Cu at (100.3, 129.0)
- added R151: 499, Resistor_SMD:R_0603_1608Metric, F.Cu at (100.3, 133.0)
- added R152: 1k, Resistor_SMD:R_0603_1608Metric, F.Cu at (93.2, 137.4)
- added R153: 1k, Resistor_SMD:R_0603_1608Metric, F.Cu at (98.2, 129.0)
- added R154: 22, Resistor_SMD:R_0603_1608Metric, F.Cu at (86.2, 132.5)
- added R155: RB, Resistor_SMD:R_0603_1608Metric, F.Cu at (42.0, 52.0)
- added R156: RB, Resistor_SMD:R_0603_1608Metric, F.Cu at (37.1, 52.4)
- added R157: RB, Resistor_SMD:R_0603_1608Metric, F.Cu at (32.1, 54.8)
- added R158: RB, Resistor_SMD:R_0603_1608Metric, F.Cu at (42.0, 65.5)
- added R159: RB, Resistor_SMD:R_0603_1608Metric, F.Cu at (37.4, 65.3)
- added R160: RB, Resistor_SMD:R_0603_1608Metric, F.Cu at (32.3, 64.5)
- added R161: 1k, Resistor_SMD:R_0603_1608Metric, F.Cu at (47.3, 58.1)
- added R162: 1k, Resistor_SMD:R_0603_1608Metric, F.Cu at (47.3, 53.6)
- added R163: 1k, Resistor_SMD:R_0603_1608Metric, F.Cu at (47.3, 49.3)
- added R164: 1k, Resistor_SMD:R_0603_1608Metric, F.Cu at (47.3, 70.8)
- added R165: 1k, Resistor_SMD:R_0603_1608Metric, F.Cu at (47.3, 66.6)
- added R166: 1k, Resistor_SMD:R_0603_1608Metric, F.Cu at (47.3, 62.6)
- added R167: 499, Resistor_SMD:R_0603_1608Metric, F.Cu at (51.1, 58.1)
- added R168: 499, Resistor_SMD:R_0603_1608Metric, F.Cu at (51.1, 53.6)
- added R169: 499, Resistor_SMD:R_0603_1608Metric, F.Cu at (51.1, 49.3)
- added R170: 499, Resistor_SMD:R_0603_1608Metric, F.Cu at (51.1, 70.8)
- added R171: 499, Resistor_SMD:R_0603_1608Metric, F.Cu at (51.1, 66.6)
- added R172: 499, Resistor_SMD:R_0603_1608Metric, F.Cu at (51.1, 62.6)
- added R173: 1k, Resistor_SMD:R_0603_1608Metric, F.Cu at (58.3, 58.2)
- added R174: 1k, Resistor_SMD:R_0603_1608Metric, F.Cu at (53.3, 66.6)
- added R175: 22, Resistor_SMD:R_0603_1608Metric, F.Cu at (65.2, 63.1)
- added U10: ~, Package_DFN_QFN:QFN-40-1EP_6x6mm_P0.5mm_EP4.6x4.6mm, F.Cu at (60.2, 64.8)
- added U9: ~, Package_DFN_QFN:QFN-40-1EP_6x6mm_P0.5mm_EP4.6x4.6mm, F.Cu at (91.2, 130.7)
- C1: value 100uF/25V -> 680uF/35V
- C18, C21, C22, C23: value 22nF -> 10nF
- C24, C47, C56, C69, C70, C83, C89: value 22nF -> 4.7uF
- C25, C43, C48, C57, C71, C90: value 22nF -> 0.22uF
- C26, C28, C29: value 4.7uF -> 10nF
- C27: value 0.1uF -> 10nF
- C30, C32: value 0.22uF -> 1uF/35V
- C31, C33: value 22nF -> 1uF/35V
- C39, C45, C52, C54, C64, C67, C77, C91, C93, C96: value 4.7uF -> 22nF
- C40, C53, C65, C81, C92: value 0.1uF -> 22nF
- C42, C55, C97: value 0.22uF -> 4.7uF
- C44, C58, C72, C86: value 22nF -> 0.1uF
- C46, C68, C78, C80, C94: value 0.22uF -> 22nF
- C76: value 4.7uF -> 0.22uF
- J1: footprint Connector_BarrelJack:BarrelJack_SwitchcraftConxall_RAPC10U_Horizontal -> Connector_BarrelJack:BarrelJack_Horizontal
- J4: value STX-4335-5BGP-S1 -> Barrel_Jack; footprint Connector_Audio:STX-4335-5BGP-S1_KYC -> Connector_BarrelJack:BarrelJack_Horizontal; moved to F.Cu
- R100, R29, R30, R32, R57, R73, R74, R75, R76, R77, R78, R94, R95, R96, R99: value 1k -> 499
- R101, R31, R34, R35: value 22 -> 499
- R102, R103, R114, R115, R116, R47, R50, R51, R67, R79: value 22 -> 1k
- R104, R81: value RB -> 22
- R109, R110, R41, R42, R43, R44, R45, R61, R62, R64: value 1k -> RB
- R17, R20, R21, R22: value RB -> 75
- R18, R19: value 22 -> 75
- R23: value RB -> 2.2K
- R24: value RB -> 2.2k
- R25, R26, R27, R28: value 1k -> 21.5K
- R33, R36, R37, R38, R52, R53, R54, R55, R56: value RB -> 499
- R39, R49, R68, R69, R70, R71, R72, R88, R89: value RB -> 1k
- R60: value 1k -> 22
- R63, R66, R82, R83: value 22 -> RB
- SW5: value SW_MEC_5E -> RotaryEncoder; footprint Button_Switch_SMD:SW_Push_1P1T_NO_6x6mm_H13mm -> Rotary_Encoder:RotaryEncoder_Alps_EC12E_Vertical_H20mm
- U2, U4, U5, U6, U7: footprint emon36:QFN50P600X600X75-41N-D -> Package_DFN_QFN:QFN-40-1EP_6x6mm_P0.5mm_EP4.6x4.6mm
- U3: value ~ -> 16.384MHz; footprint emon36:QFN50P600X600X75-41N-D -> Oscillator:Oscillator_SMD_Kyocera_KC2520Z-4Pin_2.5x2.0mm
- moved C7 232.1 mm to (-31.3, 129.4)
- moved C18 174.9 mm to (223.3, 111.5)
- moved C22 174.9 mm to (223.1, 103.7)
- moved C23 174.9 mm to (223.1, 101.1)
- moved C24 174.9 mm to (223.1, 120.4)
- moved C26 174.9 mm to (223.1, 106.8)
- moved C28 174.9 mm to (236.6, 117.2)
- moved C29 174.9 mm to (225.7, 116.6)
- moved C3 174.9 mm to (252.7, 92.7)
- moved C31 174.9 mm to (237.9, 121.7)
- moved C33 174.9 mm to (235.8, 111.5)
- moved C4 174.9 mm to (253.3, 83.9)
- moved C5 174.9 mm to (253.5, 85.8)
- moved C6 174.9 mm to (252.9, 98.7)
- moved R17 174.9 mm to (217.4, 110.9)
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Connections:
- C10 pad 2: GND -> /CH1/IDEF_N
- C11 pad 2: GND -> /CH1/IDEF_N
- C12 pad 2: GND -> /CH1/IDEF_N
- C15 pad 1: Net-(C15-Pad1) -> Net-(R16-Pad2)
- C18 pad 1: /CH2/IA_P -> Net-(C18-Pad1)
- C2 pad 2: GND -> /CH1/IABC_N
- C21 pad 1: /CH2/IB_P -> Net-(C18-Pad1)
- C22 pad 1: /CH2/IC_P -> Net-(C18-Pad1)
- C23 pad 1: /CH2/ID_P -> Net-(C18-Pad1)
- C24 pad 1: /CH2/IE_P -> 3V3
- C25 pad 1: /CH2/IF_P -> 3V3
- C26 pad 1: Net-(C26-Pad1) -> Net-(R117-Pad2)
- C27 pad 1: Net-(C26-Pad1) -> Net-(R118-Pad2)
- C29 pad 1: Net-(C29-Pad1) -> /RESET
- C3 pad 1: Net-(C1-Pad1) -> Net-(C3-Pad1)
- C30 pad 1: Net-(C29-Pad1) -> Net-(C30-Pad1)
- C30 pad 2: GND -> Net-(C30-Pad2)
- C31 pad 2: GND -> Net-(C31-Pad2)
- C32 pad 1: Net-(C28-Pad1) -> Net-(C32-Pad1)
- C32 pad 2: GND -> Net-(C32-Pad2)
- C33 pad 1: /CH3/IB_P -> Net-(C33-Pad1)
- C33 pad 2: GND -> Net-(C33-Pad2)
- C34 pad 1: /CH3/IA_P -> Net-(U2-Pad12)
- C35 pad 1: /CH3/IC_P -> /CH2/IA_P
- C35 pad 2: GND -> /CH2/IABC_N
- C36 pad 1: /CH3/ID_P -> /CH2/IB_P
- C36 pad 2: GND -> /CH2/IABC_N
- C37 pad 1: /CH3/IE_P -> /CH2/IC_P
- C37 pad 2: GND -> /CH2/IABC_N
- C38 pad 1: /CH3/IF_P -> /CH2/ID_P
- C38 pad 2: GND -> /CH2/IDEF_N
- C39 pad 1: Net-(C39-Pad1) -> /CH2/IE_P
- C39 pad 2: GND -> /CH2/IDEF_N
- C40 pad 1: Net-(C39-Pad1) -> /CH2/IF_P
- C40 pad 2: GND -> /CH2/IDEF_N
- C42 pad 1: Net-(C41-Pad1) -> Net-(C42-Pad1)
- C43 pad 1: /CH4/IB_P -> Net-(C41-Pad1)
- C44 pad 1: /CH4/IC_P -> Net-(C42-Pad1)
- C46 pad 1: Net-(C45-Pad1) -> Net-(C46-Pad1)
- C48 pad 1: /CH4/ID_P -> Net-(C47-Pad1)
- C49 pad 1: /CH4/IE_P -> /CH3/IA_P
- C49 pad 2: GND -> /CH3/IABC_N
- C50 pad 1: /CH4/IA_P -> /CH3/IB_P
- C50 pad 2: GND -> /CH3/IABC_N
- C51 pad 1: /CH4/IF_P -> /CH3/IC_P
- C51 pad 2: GND -> /CH3/IABC_N
- C52 pad 1: Net-(C52-Pad1) -> /CH3/ID_P
- C52 pad 2: GND -> /CH3/IDEF_N
- C53 pad 1: Net-(C52-Pad1) -> /CH3/IE_P
- C53 pad 2: GND -> /CH3/IDEF_N
- C54 pad 1: Net-(C54-Pad1) -> /CH3/IF_P
- C54 pad 2: GND -> /CH3/IDEF_N
- C55 pad 1: Net-(C54-Pad1) -> Net-(C55-Pad1)
- C56 pad 1: /CH5/IB_P -> Net-(C56-Pad1)
- C57 pad 1: /CH5/IC_P -> Net-(C55-Pad1)
- C58 pad 1: /CH5/ID_P -> Net-(C56-Pad1)
- C59 pad 1: /CH5/IE_P -> Net-(C59-Pad1)
- C60 pad 1: /CH5/IF_P -> Net-(C60-Pad1)
- C63 pad 1: Net-(C63-Pad1) -> /CH4/IA_P
- C63 pad 2: GND -> /CH4/IABC_N
- C64 pad 1: Net-(C64-Pad1) -> /CH4/IB_P
- C64 pad 2: GND -> /CH4/IABC_N
- C65 pad 1: Net-(C64-Pad1) -> /CH4/IC_P
- C65 pad 2: GND -> /CH4/IABC_N
- C66 pad 1: /CH5/IA_P -> /CH4/ID_P
- C66 pad 2: GND -> /CH4/IDEF_N
- C67 pad 1: Net-(C67-Pad1) -> /CH4/IE_P
- C67 pad 2: GND -> /CH4/IDEF_N
- C68 pad 1: Net-(C67-Pad1) -> /CH4/IF_P
- C68 pad 2: GND -> /CH4/IDEF_N
- C69 pad 1: /CH7/IA_P -> Net-(C69-Pad1)
- C70 pad 1: /CH7/IB_P -> Net-(C70-Pad1)
- C71 pad 1: /CH7/IC_P -> Net-(C69-Pad1)
- C72 pad 1: /CH7/ID_P -> Net-(C70-Pad1)
- C73 pad 1: /CH7/IE_P -> Net-(C73-Pad1)
- C74 pad 1: /CH7/IF_P -> Net-(C74-Pad1)
- C76 pad 1: Net-(C76-Pad1) -> Net-(C75-Pad1)
- C77 pad 1: Net-(C77-Pad1) -> /CH5/IA_P
- C77 pad 2: GND -> /CH5/IABC_N
- C78 pad 1: Net-(C77-Pad1) -> /CH5/IB_P
- C78 pad 2: GND -> /CH5/IABC_N
- C79 pad 1: Net-(C79-Pad1) -> /CH5/IC_P
- C79 pad 2: GND -> /CH5/IABC_N
- C8 pad 2: GND -> /CH1/IABC_N
- C80 pad 1: Net-(C75-Pad1) -> /CH5/ID_P
- C80 pad 2: GND -> /CH5/IDEF_N
- C81 pad 1: Net-(C76-Pad1) -> /CH5/IE_P
- C81 pad 2: GND -> /CH5/IDEF_N
- C82 pad 1: /CH0/IA_P -> /CH5/IF_P
- C82 pad 2: GND -> /CH5/IDEF_N
- C85 pad 1: Net-(C84-Pad1) -> Net-(C83-Pad1)
- C86 pad 1: /CH0/IB_P -> Net-(C84-Pad1)
- C87 pad 1: /CH0/IC_P -> Net-(C87-Pad1)
- C88 pad 1: /CH0/ID_P -> Net-(C88-Pad1)
- C89 pad 1: /CH0/IE_P -> Net-(C89-Pad1)
- C9 pad 2: GND -> /CH1/IABC_N
- C90 pad 1: /CH0/IF_P -> Net-(C89-Pad1)
- C91 pad 1: Net-(C91-Pad1) -> /CH6/IA_P
- C91 pad 2: GND -> /CH6/IABC_N
- C92 pad 1: Net-(C91-Pad1) -> /CH6/IB_P
- C92 pad 2: GND -> /CH6/IABC_N
- C93 pad 1: Net-(C93-Pad1) -> /CH6/IC_P
- C93 pad 2: GND -> /CH6/IABC_N
- C94 pad 1: Net-(C93-Pad1) -> /CH6/ID_P
- C94 pad 2: GND -> /CH6/IDEF_N
- C95 pad 1: Net-(C95-Pad1) -> /CH6/IE_P
- C95 pad 2: GND -> /CH6/IDEF_N
- C96 pad 1: Net-(C96-Pad1) -> /CH6/IF_P
- C96 pad 2: GND -> /CH6/IDEF_N
- C97 pad 1: Net-(C96-Pad1) -> Net-(C101-Pad1)
- D1 pad 2: GND -> Net-(D1-Pad2)
- D1 pad 3: Net-(D1-Pad3) -> Net-(C31-Pad1)
- D1 pad 4: Net-(D1-Pad4) -> Net-(C30-Pad2)
- D3 pad 1: unconnected-(D3-Pad1) -> Net-(C3-Pad1)
- D3 pad 2: unconnected-(D3-Pad2) -> Net-(C1-Pad1)
- J1 pad 1: Net-(D1-Pad4) -> Net-(C30-Pad2)
- J1 pad 2: Net-(D1-Pad3) -> Net-(C31-Pad1)
- J10 pad 1: GND -> /CH4/IDEF_N
- J11 pad 1: GND -> /CH5/IABC_N
- J12 pad 1: GND -> /CH5/IDEF_N
- J13 pad 1: GND -> /CH6/IABC_N
- J14 pad 1: GND -> /CH6/IDEF_N
- J15 pad 1: GND -> /CH0/IABC_N
- J2 pad 1: GND -> /CH1/IABC_N
- J3 pad 1: GND -> /CH1/IDEF_N
- J4 pad 1: GND -> Net-(C32-Pad2)
- J4 pad 2: unconnected-(J4-Pad2) -> Net-(C33-Pad1)
- J5 pad 1: GND -> /CH2/IABC_N
- J6 pad 1: GND -> /CH2/IDEF_N
- J7 pad 1: GND -> /CH3/IABC_N
- J8 pad 1: GND -> /CH3/IDEF_N
- J9 pad 1: GND -> /CH4/IABC_N
- R1 pad 2: GND -> /CH1/IABC_N
- R100 pad 1: GND -> /CH4/IE_P
- R100 pad 2: Net-(C83-Pad1) -> /CH4/IDEF_N
- R101 pad 1: Net-(R101-Pad1) -> /CH4/IF_P
- R101 pad 2: /MISO -> /CH4/IDEF_N
- R102 pad 1: Net-(R102-Pad1) -> GND
- R102 pad 2: /CH7/IRQ -> Net-(C73-Pad1)
- R103 pad 1: Net-(R103-Pad1) -> GND
- R103 pad 2: /CH7/IRQ -> Net-(C74-Pad1)
- R104 pad 1: Net-(J14-Pad25) -> Net-(R104-Pad1)
- R104 pad 2: GND -> /SPI_MISO
- R105 pad 1: Net-(J14-Pad5) -> Net-(J11-Pad35)
- R105 pad 2: GND -> /CH5/IABC_N
- R106 pad 1: Net-(J15-Pad35) -> Net-(J11-Pad25)
- R106 pad 2: GND -> /CH5/IABC_N
- R107 pad 1: Net-(J15-Pad25) -> Net-(J11-Pad5)
- R107 pad 2: GND -> /CH5/IABC_N
- R108 pad 1: Net-(J15-Pad5) -> Net-(J12-Pad35)
- R108 pad 2: GND -> /CH5/IDEF_N
- R109 pad 1: Net-(J14-Pad25) -> Net-(J12-Pad25)
- R109 pad 2: /CH0/IB_P -> /CH5/IDEF_N
- R110 pad 1: Net-(J14-Pad5) -> Net-(J12-Pad5)
- R110 pad 2: /CH0/IC_P -> /CH5/IDEF_N
- R111 pad 1: Net-(J15-Pad35) -> Net-(J11-Pad35)
- R111 pad 2: /CH0/ID_P -> /CH5/IA_P
- R112 pad 1: Net-(J15-Pad25) -> Net-(J11-Pad25)
- R112 pad 2: /CH0/IE_P -> /CH5/IB_P
- R113 pad 1: Net-(J15-Pad5) -> Net-(J11-Pad5)
- R113 pad 2: /CH0/IF_P -> /CH5/IC_P
- R114 pad 1: Net-(R114-Pad1) -> Net-(J12-Pad35)
- R114 pad 2: /MISO -> /CH5/ID_P
- R115 pad 1: Net-(R115-Pad1) -> Net-(J12-Pad25)
- R115 pad 2: /CH0/IRQ -> /CH5/IE_P
- R116 pad 1: Net-(R116-Pad1) -> Net-(J12-Pad5)
- R116 pad 2: /CH0/IRQ -> /CH5/IF_P
- R117 pad 2: GND -> Net-(R117-Pad2)
- R118 pad 2: GND -> Net-(R118-Pad2)
- R15 pad 2: /MISO -> /SPI_MISO
- R16 pad 2: Net-(C15-Pad1) -> Net-(R16-Pad2)
- R17 pad 1: Net-(J4-Pad35) -> /CLK16MHZ
- R17 pad 2: GND -> Net-(C18-Pad1)
- R18 pad 1: Net-(R18-Pad1) -> /CLK16MHZ
- R18 pad 2: /CH1/IRQ -> Net-(C18-Pad1)
- R19 pad 1: Net-(R19-Pad1) -> /CLK16MHZ
- R19 pad 2: /CH1/IRQ -> Net-(C18-Pad1)
- R20 pad 1: Net-(J4-Pad25) -> /CLK16MHZ
- R20 pad 2: GND -> Net-(C18-Pad1)
- R21 pad 1: Net-(J4-Pad5) -> Net-(R21-Pad1)
- R21 pad 2: GND -> /CLK16MHZ
- R22 pad 1: Net-(J5-Pad35) -> /SPI_MISO
- R22 pad 2: GND -> Net-(C28-Pad1)
- R23 pad 1: Net-(J5-Pad25) -> 3V3
- R23 pad 2: GND -> /RESET
- R24 pad 1: Net-(J5-Pad5) -> /SPI_CS6
- R24 pad 2: GND -> /IRQ
- R25 pad 1: Net-(J4-Pad25) -> Net-(C30-Pad1)
- R25 pad 2: /CH2/IB_P -> /VA+
- R26 pad 1: Net-(J4-Pad35) -> Net-(C31-Pad2)
- R26 pad 2: /CH2/IA_P -> /VA-
- R27 pad 1: Net-(J4-Pad5) -> Net-(C32-Pad1)
- R27 pad 2: /CH2/IC_P -> /VBI+
- R28 pad 1: Net-(J5-Pad35) -> Net-(C33-Pad2)
- R28 pad 2: /CH2/ID_P -> /VBI-
- R29 pad 1: Net-(J5-Pad25) -> /VA+
- R29 pad 2: /CH2/IE_P -> GND
- R30 pad 1: Net-(J5-Pad5) -> GND
- R30 pad 2: /CH2/IF_P -> /VA-
- R31 pad 1: Net-(R31-Pad1) -> /VBI+
- R31 pad 2: /MISO -> GND
- R32 pad 2: Net-(C31-Pad1) -> /VBI-
- R33 pad 1: Net-(J6-Pad35) -> /CH1/IA_P
- R33 pad 2: GND -> /CH1/IABC_N
- R34 pad 1: Net-(R34-Pad1) -> /CH1/IB_P
- R34 pad 2: /CH2/IRQ -> /CH1/IABC_N
- R35 pad 1: Net-(R35-Pad1) -> /CH1/IC_P
- R35 pad 2: /CH2/IRQ -> /CH1/IABC_N
- R36 pad 1: Net-(J6-Pad25) -> /CH1/ID_P
- R36 pad 2: GND -> /CH1/IDEF_N
- R37 pad 1: Net-(J6-Pad5) -> /CH1/IE_P
- R37 pad 2: GND -> /CH1/IDEF_N
- R38 pad 1: Net-(J7-Pad35) -> /CH1/IF_P
- R38 pad 2: GND -> /CH1/IDEF_N
- R39 pad 1: Net-(J7-Pad25) -> GND
- R39 pad 2: GND -> Net-(U2-Pad12)
- R4 pad 2: GND -> /CH1/IABC_N
- R40 pad 1: Net-(J7-Pad5) -> Net-(J5-Pad35)
- R40 pad 2: GND -> /CH2/IABC_N
- R41 pad 1: Net-(J6-Pad25) -> Net-(J5-Pad25)
- R41 pad 2: /CH3/IB_P -> /CH2/IABC_N
- R42 pad 1: Net-(J6-Pad35) -> Net-(J5-Pad5)
- R42 pad 2: /CH3/IA_P -> /CH2/IABC_N
- R43 pad 1: Net-(J6-Pad5) -> Net-(J6-Pad35)
- R43 pad 2: /CH3/IC_P -> /CH2/IDEF_N
- R44 pad 1: Net-(J7-Pad35) -> Net-(J6-Pad25)
- R44 pad 2: /CH3/ID_P -> /CH2/IDEF_N
- R45 pad 1: Net-(J7-Pad25) -> Net-(J6-Pad5)
- R45 pad 2: /CH3/IE_P -> /CH2/IDEF_N
- R46 pad 1: Net-(J7-Pad5) -> Net-(J5-Pad35)
- R46 pad 2: /CH3/IF_P -> /CH2/IA_P
- R47 pad 1: Net-(R47-Pad1) -> Net-(J5-Pad25)
- R47 pad 2: /MISO -> /CH2/IB_P
- R48 pad 1: GND -> Net-(J5-Pad5)
- R48 pad 2: Net-(C47-Pad1) -> /CH2/IC_P
- R49 pad 1: Net-(J8-Pad35) -> Net-(J6-Pad35)
- R49 pad 2: GND -> /CH2/ID_P
- R5 pad 2: GND -> /CH1/IABC_N
- R50 pad 1: Net-(R50-Pad1) -> Net-(J6-Pad25)
- R50 pad 2: /CH3/IRQ -> /CH2/IE_P
- R51 pad 1: Net-(R51-Pad1) -> Net-(J6-Pad5)
- R51 pad 2: /CH3/IRQ -> /CH2/IF_P
- R52 pad 1: Net-(J8-Pad25) -> /CH2/IA_P
- R52 pad 2: GND -> /CH2/IABC_N
- R53 pad 1: Net-(J8-Pad5) -> /CH2/IB_P
- R53 pad 2: GND -> /CH2/IABC_N
- R54 pad 1: Net-(J9-Pad35) -> /CH2/IC_P
- R54 pad 2: GND -> /CH2/IABC_N
- R55 pad 1: Net-(J9-Pad25) -> /CH2/ID_P
- R55 pad 2: GND -> /CH2/IDEF_N
- R56 pad 1: Net-(J9-Pad5) -> /CH2/IE_P
- R56 pad 2: GND -> /CH2/IDEF_N
- R57 pad 1: Net-(J8-Pad25) -> /CH2/IF_P
- R57 pad 2: /CH4/IB_P -> /CH2/IDEF_N
- R58 pad 1: Net-(J8-Pad35) -> GND
- R58 pad 2: /CH4/IA_P -> Net-(C45-Pad1)
- R59 pad 1: Net-(J8-Pad5) -> GND
- R59 pad 2: /CH4/IC_P -> Net-(C46-Pad1)
- R6 pad 2: GND -> /CH1/IDEF_N
- R60 pad 1: Net-(J9-Pad35) -> Net-(R60-Pad1)
- R60 pad 2: /CH4/ID_P -> /SPI_MISO
- R61 pad 1: Net-(J9-Pad25) -> Net-(J7-Pad35)
- R61 pad 2: /CH4/IE_P -> /CH3/IABC_N
- R62 pad 1: Net-(J9-Pad5) -> Net-(J7-Pad25)
- R62 pad 2: /CH4/IF_P -> /CH3/IABC_N
- R63 pad 1: Net-(R63-Pad1) -> Net-(J7-Pad5)
- R63 pad 2: /MISO -> /CH3/IABC_N
- R64 pad 1: GND -> Net-(J8-Pad35)
- R64 pad 2: Net-(C63-Pad1) -> /CH3/IDEF_N
- R65 pad 1: Net-(J10-Pad35) -> Net-(J8-Pad25)
- R65 pad 2: GND -> /CH3/IDEF_N
- R66 pad 1: Net-(R66-Pad1) -> Net-(J8-Pad5)
- R66 pad 2: /CH4/IRQ -> /CH3/IDEF_N
- R67 pad 1: Net-(R67-Pad1) -> Net-(J7-Pad35)
- R67 pad 2: /CH4/IRQ -> /CH3/IA_P
- R68 pad 1: Net-(J10-Pad25) -> Net-(J7-Pad25)
- R68 pad 2: GND -> /CH3/IB_P
- R69 pad 1: Net-(J10-Pad5) -> Net-(J7-Pad5)
- R69 pad 2: GND -> /CH3/IC_P
- R7 pad 2: GND -> /CH1/IDEF_N
- R70 pad 1: Net-(J11-Pad35) -> Net-(J8-Pad35)
- R70 pad 2: GND -> /CH3/ID_P
- R71 pad 1: Net-(J11-Pad25) -> Net-(J8-Pad25)
- R71 pad 2: GND -> /CH3/IE_P
- R72 pad 1: Net-(J11-Pad5) -> Net-(J8-Pad5)
- R72 pad 2: GND -> /CH3/IF_P
- R73 pad 1: Net-(J10-Pad25) -> /CH3/IA_P
- R73 pad 2: /CH5/IB_P -> /CH3/IABC_N
- R74 pad 1: Net-(J10-Pad35) -> /CH3/IB_P
- R74 pad 2: /CH5/IA_P -> /CH3/IABC_N
- R75 pad 1: Net-(J10-Pad5) -> /CH3/IC_P
- R75 pad 2: /CH5/IC_P -> /CH3/IABC_N
- R76 pad 1: Net-(J11-Pad35) -> /CH3/ID_P
- R76 pad 2: /CH5/ID_P -> /CH3/IDEF_N
- R77 pad 1: Net-(J11-Pad25) -> /CH3/IE_P
- R77 pad 2: /CH5/IE_P -> /CH3/IDEF_N
- R78 pad 1: Net-(J11-Pad5) -> /CH3/IF_P
- R78 pad 2: /CH5/IF_P -> /CH3/IDEF_N
- R79 pad 1: Net-(R79-Pad1) -> GND
- R79 pad 2: /MISO -> Net-(C59-Pad1)
- R8 pad 2: GND -> /CH1/IDEF_N
- R80 pad 2: Net-(C79-Pad1) -> Net-(C60-Pad1)
- R81 pad 1: Net-(J14-Pad35) -> Net-(R81-Pad1)
- R81 pad 2: GND -> /SPI_MISO
- R82 pad 1: Net-(R82-Pad1) -> Net-(J9-Pad35)
- R82 pad 2: /CH5/IRQ -> /CH4/IABC_N
- R83 pad 1: Net-(R83-Pad1) -> Net-(J9-Pad25)
- R83 pad 2: /CH5/IRQ -> /CH4/IABC_N
- R84 pad 1: Net-(J12-Pad35) -> Net-(J9-Pad5)
- R84 pad 2: GND -> /CH4/IABC_N
- R85 pad 1: Net-(J12-Pad25) -> Net-(J10-Pad35)
- R85 pad 2: GND -> /CH4/IDEF_N
- R86 pad 1: Net-(J12-Pad5) -> Net-(J10-Pad25)
- R86 pad 2: GND -> /CH4/IDEF_N
- R87 pad 1: Net-(J13-Pad35) -> Net-(J10-Pad5)
- R87 pad 2: GND -> /CH4/IDEF_N
- R88 pad 1: Net-(J13-Pad25) -> Net-(J9-Pad35)
- R88 pad 2: GND -> /CH4/IA_P
- R89 pad 1: Net-(J13-Pad5) -> Net-(J9-Pad25)
- R89 pad 2: GND -> /CH4/IB_P
- R90 pad 1: Net-(J14-Pad35) -> Net-(J9-Pad5)
- R90 pad 2: /CH0/IA_P -> /CH4/IC_P
- R91 pad 1: Net-(J12-Pad35) -> Net-(J10-Pad35)
- R91 pad 2: /CH7/IA_P -> /CH4/ID_P
- R92 pad 1: Net-(J12-Pad25) -> Net-(J10-Pad25)
- R92 pad 2: /CH7/IB_P -> /CH4/IE_P
- R93 pad 1: Net-(J12-Pad5) -> Net-(J10-Pad5)
- R93 pad 2: /CH7/IC_P -> /CH4/IF_P
- R94 pad 1: Net-(J13-Pad35) -> /CH4/IA_P
- R94 pad 2: /CH7/ID_P -> /CH4/IABC_N
- R95 pad 1: Net-(J13-Pad25) -> /CH4/IB_P
- R95 pad 2: /CH7/IE_P -> /CH4/IABC_N
- R96 pad 1: GND -> /CH4/IC_P
- R96 pad 2: Net-(C95-Pad1) -> /CH4/IABC_N
- R99 pad 1: Net-(J13-Pad5) -> /CH4/ID_P
- R99 pad 2: /CH7/IF_P -> /CH4/IDEF_N
- U1 pad 2: unconnected-(U1-Pad2) -> /RESET
- U1 pad 5: /SCLK -> /SPI_SCLK
- U2 pad 12: Net-(C15-Pad1) -> Net-(U2-Pad12)
- U2 pad 14: Net-(C15-Pad1) -> Net-(U2-Pad12)
- U2 pad 15: unconnected-(U2-Pad15) -> /VA+
- U2 pad 16: Net-(C15-Pad1) -> /VA-
- U2 pad 18: Net-(C15-Pad1) -> Net-(R16-Pad2)
- U2 pad 27: /CH1/CLKIN -> /CLK16MHZ
- U2 pad 29: Net-(R19-Pad1) -> /IRQ
- U2 pad 32: Net-(R18-Pad1) -> /IRQ
- U2 pad 4: /CH1/RESET -> /RESET
- U2 pad 8: Net-(C15-Pad1) -> Net-(U2-Pad12)
- U3 pad 1: GND -> unconnected-(U3-Pad1)
- U3 pad 2: 3V3 -> GND
- U3 pad 3: GND -> Net-(R21-Pad1)
- U3 pad 4: /CH2/RESET -> 3V3
- U4 pad 12: Net-(C47-Pad1) -> Net-(C45-Pad1)
- U4 pad 13: /CH3/IC_P -> /CH2/IC_P
- U4 pad 14: Net-(C47-Pad1) -> Net-(C45-Pad1)
- U4 pad 15: unconnected-(U4-Pad15) -> /VA+
- U4 pad 16: Net-(C47-Pad1) -> /VA-
- U4 pad 17: Net-(C39-Pad1) -> Net-(C42-Pad1)
- U4 pad 18: Net-(C47-Pad1) -> Net-(C46-Pad1)
- U4 pad 19: /CH3/IF_P -> /CH2/IF_P
- U4 pad 22: /CH3/IE_P -> /CH2/IE_P
- U4 pad 23: /CH3/ID_P -> /CH2/ID_P
- U4 pad 24: Net-(C45-Pad1) -> Net-(C41-Pad1)
- U4 pad 27: /CH3/CLKIN -> /CLK16MHZ
- U4 pad 29: Net-(R51-Pad1) -> /IRQ
- U4 pad 32: Net-(R50-Pad1) -> /IRQ
- U4 pad 37: Net-(R47-Pad1) -> Net-(R60-Pad1)
- U4 pad 39: /SPI_CS3 -> /SPI_CS2
- U4 pad 4: /CH3/RESET -> /RESET
- U4 pad 5: Net-(C41-Pad1) -> Net-(C47-Pad1)
- U4 pad 7: /CH3/IA_P -> /CH2/IA_P
- U4 pad 8: Net-(C47-Pad1) -> Net-(C45-Pad1)
- U4 pad 9: /CH3/IB_P -> /CH2/IB_P
- U5 pad 12: Net-(C63-Pad1) -> Net-(C59-Pad1)
- U5 pad 13: /CH4/IC_P -> /CH3/IC_P
- U5 pad 14: Net-(C63-Pad1) -> Net-(C59-Pad1)
- U5 pad 15: unconnected-(U5-Pad15) -> /VA+
- U5 pad 16: Net-(C63-Pad1) -> /VA-
- U5 pad 17: Net-(C52-Pad1) -> Net-(C56-Pad1)
- U5 pad 18: Net-(C63-Pad1) -> Net-(C60-Pad1)
- U5 pad 19: /CH4/IF_P -> /CH3/IF_P
- U5 pad 22: /CH4/IE_P -> /CH3/IE_P
- U5 pad 23: /CH4/ID_P -> /CH3/ID_P
- U5 pad 24: Net-(C61-Pad1) -> Net-(C55-Pad1)
- U5 pad 27: /CH4/CLKIN -> /CLK16MHZ
- U5 pad 29: Net-(R67-Pad1) -> /IRQ
- U5 pad 32: Net-(R66-Pad1) -> /IRQ
- U5 pad 37: Net-(R63-Pad1) -> Net-(R81-Pad1)
- U5 pad 39: /SPI_CS4 -> /SPI_CS3
- U5 pad 4: /CH4/RESET -> /RESET
- U5 pad 5: Net-(C54-Pad1) -> Net-(C61-Pad1)
- U5 pad 7: /CH4/IA_P -> /CH3/IA_P
- U5 pad 8: Net-(C63-Pad1) -> Net-(C59-Pad1)
- U5 pad 9: /CH4/IB_P -> /CH3/IB_P
- U6 pad 12: Net-(C79-Pad1) -> Net-(C73-Pad1)
- U6 pad 13: /CH5/IC_P -> /CH4/IC_P
- U6 pad 14: Net-(C79-Pad1) -> Net-(C73-Pad1)
- U6 pad 15: unconnected-(U6-Pad15) -> /VB+
- U6 pad 16: Net-(C79-Pad1) -> /VB-
- U6 pad 17: Net-(C64-Pad1) -> Net-(C70-Pad1)
- U6 pad 18: Net-(C79-Pad1) -> Net-(C74-Pad1)
- U6 pad 19: /CH5/IF_P -> /CH4/IF_P
- U6 pad 22: /CH5/IE_P -> /CH4/IE_P
- U6 pad 23: /CH5/ID_P -> /CH4/ID_P
- U6 pad 24: Net-(C77-Pad1) -> Net-(C69-Pad1)
- U6 pad 27: /CH5/CLKIN -> /CLK16MHZ
- U6 pad 29: Net-(R83-Pad1) -> /IRQ
- U6 pad 32: Net-(R82-Pad1) -> /IRQ
- U6 pad 37: Net-(R79-Pad1) -> Net-(R104-Pad1)
- U6 pad 39: /SPI_CS5 -> /SPI_CS4
- U6 pad 4: /CH5/RESET -> /CH4/RESET
- U6 pad 5: Net-(C67-Pad1) -> Net-(C75-Pad1)
- U6 pad 7: /CH5/IA_P -> /CH4/IA_P
- U6 pad 8: Net-(C79-Pad1) -> Net-(C73-Pad1)
- U6 pad 9: /CH5/IB_P -> /CH4/IB_P
- U7 pad 12: Net-(C95-Pad1) -> Net-(C87-Pad1)
- U7 pad 13: /CH0/IC_P -> /CH5/IC_P
- U7 pad 14: Net-(C95-Pad1) -> Net-(C87-Pad1)
- U7 pad 15: unconnected-(U7-Pad15) -> /VB+
- U7 pad 16: Net-(C95-Pad1) -> /VB-
- U7 pad 17: Net-(C91-Pad1) -> Net-(C84-Pad1)
- U7 pad 18: Net-(C95-Pad1) -> Net-(C88-Pad1)
- U7 pad 19: /CH0/IF_P -> /CH5/IF_P
- U7 pad 22: /CH0/IE_P -> /CH5/IE_P
- U7 pad 23: /CH0/ID_P -> /CH5/ID_P
- U7 pad 24: Net-(C93-Pad1) -> Net-(C83-Pad1)
- U7 pad 27: /CH0/CLKIN -> /CLK16MHZ
- U7 pad 29: Net-(R116-Pad1) -> /IRQ
- U7 pad 32: Net-(R115-Pad1) -> /IRQ
- U7 pad 37: Net-(R114-Pad1) -> Net-(R133-Pad1)
- U7 pad 39: /SPI_CS0 -> /SPI_CS5
- U7 pad 4: /CH0/RESET -> /RESET
- U7 pad 5: Net-(C96-Pad1) -> Net-(C89-Pad1)
- U7 pad 7: /CH0/IA_P -> /CH5/IA_P
- U7 pad 8: Net-(C95-Pad1) -> Net-(C87-Pad1)
- U7 pad 9: /CH0/IB_P -> /CH5/IB_P
- U8 pad 2: Net-(C1-Pad1) -> Net-(C3-Pad1)
Routing:
- net GND: track 100.0 -> 26.4 mm, vias 18 -> 6
- net /MISO: track 4.72 -> 0.00 mm
- net Net-(C30-Pad1): track 0.00 -> 3.44 mm, vias 0 -> 1
- net /CH4/IRQ: track 3.44 -> 0.00 mm, vias 1 -> 0
- net /CH2/IRQ: track 3.44 -> 0.00 mm, vias 1 -> 0
- net /CH1/IRQ: track 3.44 -> 0.00 mm, vias 1 -> 0
- net /CH5/IRQ: track 3.44 -> 0.00 mm, vias 1 -> 0
- net /CH1/ID_P: track 3.10 -> 0.00 mm
- net Net-(C18-Pad1): track 0.00 -> 2.98 mm, vias 0 -> 1
- net Net-(J14-Pad35): track 0.00 -> 1.72 mm
- net Net-(C83-Pad1): track 1.72 -> 0.00 mm
- net Net-(C54-Pad1): track 1.72 -> 0.00 mm
- net Net-(C39-Pad1): track 1.72 -> 0.00 mm
- net /VA+: track 0.00 -> 1.72 mm
- net /RESET: track 0.00 -> 1.72 mm
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Other:
- board size 80 x 99.1 mm -> 100 x 100 mm
